File: esptt.kicad_pcb (KiCad board)
At the start: 2 copper layers, 21.3 x 43 mm, 17 parts

Commit message: tweaks
Parts:
- moved R3 0.72 mm to (146.3, 57.4)
- gave numbers to parts that had none: 1
Changed lines of the file:
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@@
     (34 B.Paste user hide)
     (35 F.Paste user)
-    (36 B.SilkS user hide)
+    (36 B.SilkS user)
     (37 F.SilkS user)
     (38 B.Mask user)
@@
     (tags "resistor 0603")
     (attr smd)
-    (fp_text reference R2 (at 0 1.4 90) (layer F.SilkS)
-      (effects (font (size 0.8 0.8) (thickness 0.1)))
+    (fp_text reference R2 (at 0 1.016 90) (layer F.SilkS)
+      (effects (font (size 0.5 0.5) (thickness 0.1)))
     )
     (fp_text value R_0603 (at 0 1.9 90) (layer F.Fab)
@@
     (tags "pin header")
     (fp_text reference TEMP (at 0 -2.3) (layer F.SilkS)
-      (effects (font (size 1 1) (thickness 0.15)))
+      (effects (font (size 0.9 0.9) (thickness 0.1)))
     )
     (fp_text value Pin_Header_Straight_1x03 (at 0 -3.1) (layer F.Fab) hide
@@
     (tags "pin header")
     (fp_text reference LIGHT (at 0 -2.3) (layer F.SilkS)
-      (effects (font (size 1 1) (thickness 0.15)))
+      (effects (font (size 0.8 0.9) (thickness 0.15)))
     )
     (fp_text value Pin_Header_Straight_1x03 (at 0 -3.1) (layer F.Fab) hide
@@
     (tags "resistor 0603")
     (attr smd)
-    (fp_text reference R1 (at 0 1.4 90) (layer F.SilkS)
-      (effects (font (size 1 1) (thickness 0.15)))
+    (fp_text reference R1 (at 0 1.016 90) (layer F.SilkS)
+      (effects (font (size 0.5 0.5) (thickness 0.1)))
     )
     (fp_text value R_0603 (at 0 1.9 90) (layer F.Fab)
@@
   )
   (module Resistors_SMD:R_0603 (layer F.Cu)
-    (at 146.812 57.912)
+    (at 146.304 57.404)
     (descr "Resistor SMD 0603, reflow soldering, Vishay (see dcrcw.pdf)")
     (tags "resistor 0603")
     (attr smd)
-    (fp_text reference "" (at 0 -1.9) (layer F.SilkS)
-      (effects (font (size 1 1) (thickness 0.15)))
+    (fp_text reference R3 (at 0 -1.016) (layer F.SilkS)
+      (effects (font (size 0.5 0.5) (thickness 0.1)))
     )
     (fp_text value R_0603 (at 0 1.9) (layer F.Fab)
@@
       (rotate (xyz 0 0 0))
     )
+    (model Resistors_SMD.3dshapes/R_0603.wrl
+      (at (xyz 0 0 0))
+      (scale (xyz 1 1 1))
+      (rotate (xyz 0 0 0))
+    )
   )
   (module Resistors_SMD:R_0603 (layer F.Cu)
@@
     (effects (font (size 0.8 0.8) (thickness 0.2)))
   )
-  (gr_text D (at 152.1 56.6) (layer F.SilkS)
-    (effects (font (size 0.8 0.8) (thickness 0.2)))
+  (gr_text D (at 151.638 56.642) (layer F.SilkS)
+    (effects (font (size 0.6 0.6) (thickness 0.1)))
   )
   (gr_text D (at 152 46) (layer F.SilkS)
     (effects (font (size 0.8 0.8) (thickness 0.2)))
   )
-  (gr_text G (at 152.1 53.8) (layer F.SilkS)
-    (effects (font (size 0.8 0.8) (thickness 0.2)))
+  (gr_text G (at 151.638 54.102) (layer F.SilkS)
+    (effects (font (size 0.6 0.6) (thickness 0.1)))
   )
   (gr_text G (at 152 43.6) (layer F.SilkS)
@@
     (effects (font (size 0.5 0.5) (thickness 0.125)))
   )
-  (gr_text +3 (at 152.3 51.5) (layer F.SilkS)
-    (effects (font (size 0.8 0.8) (thickness 0.2)))
+  (gr_text +3 (at 151.892 51.562) (layer F.SilkS)
+    (effects (font (size 0.6 0.6) (thickness 0.1)))
   )
   (gr_text +3 (at 152.1 40.9) (layer F.SilkS)
@@
   (via (at 137.16 55.626) (size 0.6) (drill 0.4) (layers F.Cu B.Cu) (net 0))
   (segment (start 137.668 56.134) (end 137.16 55.626) (width 0.25) (layer F.Cu) (net 0))
-  (segment (start 137.816 60.068) (end 138.3 58.786) (width 0.25) (layer F.Cu) (net 0) (status 10))
-  (segment (start 138.3 58.786) (end 137.668 58.154) (width 0.25) (layer F.Cu) (net 0) (status 20))
+  (segment (start 137.816 60.068) (end 137.795 58.801) (width 0.25) (layer F.Cu) (net 0) (status 400010))
+  (segment (start 137.795 58.801) (end 137.668 58.154) (width 0.25) (layer F.Cu) (net 0) (status 800020))
   (segment (start 135.37 56.654) (end 135.128 56.896) (width 0.25) (layer F.Cu) (net 0) (status 30))
   (segment (start 137.668 54.598) (end 135.37 54.598) (width 0.25) (layer F.Cu) (net 0) (status 30))
@@
   (segment (start 137.668 53.098) (end 138.938 53.098) (width 0.25) (layer F.Cu) (net 0) (status 10))
   (segment (start 138.938 53.098) (end 138.938 53.34) (width 0.25) (layer F.Cu) (net 0))
-  (segment (start 147.562 57.912) (end 147.078 59.956) (width 0.25) (layer F.Cu) (net 0) (status 30))
+  (segment (start 147.054 57.404) (end 147.078 59.956) (width 0.25) (layer F.Cu) (net 0) (status 30))
   (segment (start 147.078 59.956) (end 146.566 60.468) (width 0.25) (layer F.Cu) (net 0) (status 30))
   (segment (start 135.14 54.368) (end 135.128 54.356) (width 0.25) (layer F.Cu) (net 0) (status 30))
@@
   (segment (start 147.1035 59.9305) (end 146.566 60.468) (width 0.25) (layer F.Cu) (net 0) (status 30))
   (segment (start 143.616 60.068) (end 143.766 60.068) (width 0.25) (layer F.Cu) (net 0) (status 30))
-  (segment (start 143.766 60.068) (end 146.05 57.912) (width 0.25) (layer F.Cu) (net 0) (status 30))
+  (segment (start 143.766 60.068) (end 145.542 57.404) (width 0.25) (layer F.Cu) (net 0) (status 30))
   (segment (start 144.78 45.72) (end 143.4 45.4) (width 0.25) (layer F.Cu) (net 0))
   (segment (start 132.842 76.454) (end 139.7 78.994) (width 0.25) (layer B.Cu) (net 0) (status 20))
@@
   (segment (start 142.4 77.3) (end 148.9 70.6) (width 0.25) (layer B.Cu) (net 0))
   (segment (start 147 62.3) (end 140.2 62.3) (width 0.25) (layer B.Cu) (net 0))
-  (segment (start 140.2 62.3) (end 137.11 59.132) (width 0.25) (layer B.Cu) (net 0))
+  (segment (start 140.2 62.3) (end 136.906 59.182) (width 0.25) (layer B.Cu) (net 0))
   (segment (start 147.05 62.25) (end 146.566 60.468) (width 0.25) (layer F.Cu) (net 0) (status 20))
   (via (at 147 62.3) (size 0.6) (drill 0.4) (layers F.Cu B.Cu) (net 0))
@@
   (segment (start 135.382 73.406) (end 135.4 59.5) (width 0.25) (layer B.Cu) (net 0))
   (via (at 135.382 73.406) (size 0.6) (drill 0.4) (layers F.Cu B.Cu) (net 0))
-  (segment (start 134.866 75.168) (end 135.332 73.356) (width 0.25) (layer F.Cu) (net 0) (status 400010))
+  (segment (start 134.866 75.168) (end 135.332 73.356) (width 0.25) (layer F.Cu) (net 0) (status 10))
   (segment (start 135.332 73.356) (end 135.382 73.406) (width 0.25) (layer F.Cu) (net 0))
-  (segment (start 135.4 59.5) (end 137.11 59.132) (width 0.25) (layer B.Cu) (net 0))
+  (segment (start 135.4 59.5) (end 136.906 59.182) (width 0.25) (layer B.Cu) (net 0))
   (segment (start 142.24 78.634) (end 142.24 78.994) (width 0.25) (layer B.Cu) (net 0) (status 30))
   (segment (start 137.816 75.568) (end 139.192 76.454) (width 0.25) (layer F.Cu) (net 0) (status 10))
@@
   (segment (start 140.7 56.8) (end 140.7 49.24) (width 0.25) (layer B.Cu) (net 0))
   (segment (start 140.7 49.24) (end 135 46.74) (width 0.25) (layer B.Cu) (net 0) (status 20))
-  (segment (start 137.11 59.132) (end 139 58.5) (width 0.25) (layer B.Cu) (net 0))
-  (segment (start 139 58.5) (end 140.7 56.8) (width 0.25) (layer B.Cu) (net 0))
-  (segment (start 137.16 59.182) (end 137.11 59.132) (width 0.25) (layer F.Cu) (net 0))
-  (via (at 137.11 59.132) (size 0.6) (drill 0.4) (layers F.Cu B.Cu) (net 0))
-  (segment (start 134.866 60.468) (end 137.16 59.182) (width 0.25) (layer F.Cu) (net 0) (status 10))
+  (segment (start 136.906 59.182) (end 139.065 58.674) (width 0.25) (layer B.Cu) (net 0))
+  (segment (start 139.065 58.674) (end 140.7 56.8) (width 0.25) (layer B.Cu) (net 0))
+  (segment (start 136.956 59.232) (end 136.906 59.182) (width 0.25) (layer F.Cu) (net 0))
+  (via (at 136.906 59.182) (size 0.6) (drill 0.4) (layers F.Cu B.Cu) (net 0))
+  (segment (start 134.866 60.468) (end 136.956 59.232) (width 0.25) (layer F.Cu) (net 0) (status 400010))
   (segment (start 140.208 55.88) (end 140.7 56.8) (width 0.25) (layer F.Cu) (net 0))
   (via (at 140.7 56.8) (size 0.6) (drill 0.4) (layers F.Cu B.Cu) (net 0))

Commit message: start 2016-Sep. No pin5/wake
Routing:
- net (no net): track 444.2 -> 432.0 mm, vias 13 -> 12
Changed lines of the file:
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@@
     (thickness 1.6)
     (drawings 20)
-    (tracks 170)
+    (tracks 163)
     (zones 0)
     (modules 17)
@@
     (34 B.Paste user hide)
     (35 F.Paste user)
-    (36 B.SilkS user)
-    (37 F.SilkS user)
+    (36 B.SilkS user hide)
+    (37 F.SilkS user hide)
     (38 B.Mask user)
     (39 F.Mask user)
@@
   (segment (start 146.05 51.310956) (end 146.05 55.372) (width 0.25) (layer F.Cu) (net 0))
   (segment (start 146.051478 51.309478) (end 146.05 51.310956) (width 0.25) (layer F.Cu) (net 0))
-  (segment (start 142.016 69.118) (end 144.272 71.374) (width 0.25) (layer F.Cu) (net 0) (status 10))
-  (segment (start 144.272 72.874) (end 146.566 75.168) (width 0.25) (layer F.Cu) (net 0) (status 20))
-  (segment (start 144.272 71.374) (end 144.272 72.874) (width 0.25) (layer F.Cu) (net 0))
   (segment (start 142.016 66.518) (end 142.782 66.518) (width 0.25) (layer F.Cu) (net 0) (status 30))
   (segment (start 142.782 66.518) (end 147 62.3) (width 0.25) (layer F.Cu) (net 0) (status 10))
@@
   (via (at 137.16 55.626) (size 0.6) (drill 0.4) (layers F.Cu B.Cu) (net 0))
   (segment (start 137.668 56.134) (end 137.16 55.626) (width 0.25) (layer F.Cu) (net 0))
-  (segment (start 137.816 60.068) (end 137.795 58.801) (width 0.25) (layer F.Cu) (net 0) (status 400010))
-  (segment (start 137.795 58.801) (end 137.668 58.154) (width 0.25) (layer F.Cu) (net 0) (status 800020))
+  (segment (start 137.816 60.068) (end 137.795 58.801) (width 0.25) (layer F.Cu) (net 0) (status 10))
+  (segment (start 137.795 58.801) (end 137.668 58.154) (width 0.25) (layer F.Cu) (net 0) (status 20))
   (segment (start 135.37 56.654) (end 135.128 56.896) (width 0.25) (layer F.Cu) (net 0) (status 30))
   (segment (start 137.668 54.598) (end 135.37 54.598) (width 0.25) (layer F.Cu) (net 0) (status 30))
@@
   (via (at 147 62.3) (size 0.6) (drill 0.4) (layers F.Cu B.Cu) (net 0))
   (segment (start 147 62.3) (end 147.05 62.25) (width 0.25) (layer F.Cu) (net 0))
-  (segment (start 148.7 75.2) (end 146.616 75.218) (width 0.25) (layer F.Cu) (net 0) (status 20))
-  (segment (start 148.7 75.2) (end 148.65 75.15) (width 0.25) (layer F.Cu) (net 0))
-  (segment (start 148.65 75.15) (end 146.566 75.168) (width 0.25) (layer F.Cu) (net 0) (status 20))
   (segment (start 148.7 75.2) (end 148.336 78.486) (width 0.25) (layer B.Cu) (net 0))
   (segment (start 148.236 78.586) (end 148.336 78.486) (width 0.25) (layer F.Cu) (net 0))
   (via (at 148.336 78.486) (size 0.6) (drill 0.4) (layers F.Cu B.Cu) (net 0))
   (segment (start 148.236 78.586) (end 144.78 78.994) (width 0.25) (layer F.Cu) (net 0) (status 20))
-  (via (at 148.7 75.2) (size 0.6) (drill 0.4) (layers F.Cu B.Cu) (net 0))
   (segment (start 146.966 70.618) (end 146.866 70.518) (width 0.25) (layer F.Cu) (net 0) (status 30))
   (segment (start 142.24 78.994) (end 142.24 78.534) (width 0.25) (layer F.Cu) (net 0) (status 30))
@@
   (segment (start 136.956 59.232) (end 136.906 59.182) (width 0.25) (layer F.Cu) (net 0))
   (via (at 136.906 59.182) (size 0.6) (drill 0.4) (layers F.Cu B.Cu) (net 0))
-  (segment (start 134.866 60.468) (end 136.956 59.232) (width 0.25) (layer F.Cu) (net 0) (status 400010))
+  (segment (start 134.866 60.468) (end 136.956 59.232) (width 0.25) (layer F.Cu) (net 0) (status 10))
   (segment (start 140.208 55.88) (end 140.7 56.8) (width 0.25) (layer F.Cu) (net 0))
   (via (at 140.7 56.8) (size 0.6) (drill 0.4) (layers F.Cu B.Cu) (net 0))

Commit message: updated eps-06 part
Parts:
- ESP-06: footprint ESP-06 -> ESP8266:ESP-06
- renumbered REF** to ?
Changed lines of the file:
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@@
     (32 B.Adhes user)
     (33 F.Adhes user)
-    (34 B.Paste user hide)
+    (34 B.Paste user)
     (35 F.Paste user)
     (36 B.SilkS user hide)
@@
     (pad 2 smd rect (at 4.7498 0 90) (size 1.39954 2.09804) (layers F.Cu F.Paste F.Mask))
   )
-  (module ESP-06 (layer F.Cu)
-    (at 140.716 67.818 90)
-    (fp_text reference ESP-06 (at 0 0.5 90) (layer F.SilkS)
-      (effects (font (size 1 1) (thickness 0.15)))
-    )
-    (fp_text value ESP-06 (at 0 -0.5 90) (layer F.Fab) hide
-      (effects (font (size 1 1) (thickness 0.15)))
-    )
-    (fp_line (start -8.15 6.55) (end 8.15 6.55) (layer F.SilkS) (width 0.15))
-    (fp_line (start 8.15 6.55) (end 8.15 -6.55) (layer F.SilkS) (width 0.15))
-    (fp_line (start 8.15 -6.55) (end -8.15 -6.55) (layer F.SilkS) (width 0.15))
-    (fp_line (start -8.15 -6.55) (end -8.15 6.55) (layer F.SilkS) (width 0.15))
-    (pad G smd rect (at -7.35 -5.85 90) (size 2 2) (layers F.Cu F.Paste F.Mask))
-    (pad G smd rect (at 7.35 -5.85 90) (size 2 2) (layers F.Cu F.Paste F.Mask))
-    (pad G smd rect (at -7.35 5.85 90) (size 2 2) (layers F.Cu F.Paste F.Mask))
-    (pad G smd rect (at 7.35 5.85 90) (size 2 2) (layers F.Cu F.Paste F.Mask))
-    (pad GP14 smd rect (at -2.7 6.15 90) (size 1 1.2) (layers F.Cu F.Paste F.Mask))
-    (pad GP13 smd rect (at 0 6.15 90) (size 1 1.2) (layers F.Cu F.Paste F.Mask))
-    (pad GP12 smd rect (at 2.7 6.15 90) (size 1 1.2) (layers F.Cu F.Paste F.Mask))
-    (pad TX smd rect (at 0 -6.15 90) (size 1 1.2) (layers F.Cu F.Paste F.Mask))
-    (pad GP16 smd rect (at -2.7 -6.15 90) (size 1 1.2) (layers F.Cu F.Paste F.Mask))
-    (pad RX smd rect (at 2.7 -6.15 90) (size 1 1.2) (layers F.Cu F.Paste F.Mask))
-    (pad 3.3 smd rect (at -7.75 0 90) (size 1.2 1) (layers F.Cu F.Paste F.Mask))
-    (pad CHPD smd rect (at -7.75 2.9 90) (size 1.2 1) (layers F.Cu F.Paste F.Mask))
-    (pad ANT smd rect (at -7.75 -2.9 90) (size 1.2 1) (layers F.Cu F.Paste F.Mask))
-    (pad GP2 smd rect (at 7.75 0 90) (size 1.2 1) (layers F.Cu F.Paste F.Mask))
-    (pad GP0 smd rect (at 7.75 -2.9 90) (size 1.2 1) (layers F.Cu F.Paste F.Mask))
-    (pad GP15 smd rect (at 7.75 2.9 90) (size 1.2 1) (layers F.Cu F.Paste F.Mask))
-    (pad Gx smd rect (at -1.3 -1.3 90) (size 2 2) (layers F.Cu F.Paste F.Mask))
-    (pad Gx smd rect (at 1.3 -1.3 90) (size 2 2) (layers F.Cu F.Paste F.Mask))
-    (pad Gx smd rect (at -1.3 1.3 90) (size 2 2) (layers F.Cu F.Paste F.Mask))
-    (pad Gx smd rect (at 1.3 1.3 90) (size 2 2) (layers F.Cu F.Paste F.Mask))
-  )
   (module Connect:USB_Micro-B_10103594-0001LF (layer F.Cu)
     (at 142.3 41.6 180)
@@
     (tags "resistor 0603")
     (attr smd)
-    (fp_text reference REF** (at 0 -1.9 90) (layer F.SilkS)
+    (fp_text reference "" (at 0 -1.9 90) (layer F.SilkS)
       (effects (font (size 1 1) (thickness 0.15)))
     )
@@
     (pad 1 np_thru_hole circle (at 0 0) (size 2.2 2.2) (drill 2.2) (layers *.Cu *.Mask F.SilkS))
   )
+  (module ESP8266:ESP-06 (layer F.Cu)
+    (at 140.716 67.818 90)
+    (fp_text reference ESP-06 (at 0 0.5 90) (layer F.SilkS)
+      (effects (font (size 1 1) (thickness 0.15)))
+    )
+    (fp_text value ESP-06 (at 0 -0.5 90) (layer F.Fab)
+      (effects (font (size 1 1) (thickness 0.15)))
+    )
+    (fp_text user AI (at -5.65 -3.95 90) (layer F.SilkS)
+      (effects (font (size 1 1) (thickness 0.15)))
+    )
+    (fp_text user WIFI (at 4.25 -4.4 90) (layer F.SilkS)
+      (effects (font (size 1 1) (thickness 0.15)))
+    )
+    (fp_text user FCC (at -5.6 4.05 90) (layer F.SilkS)
+      (effects (font (size 1 1) (thickness 0.15)))
+    )
+    (fp_line (start -8.15 6.55) (end 8.15 6.55) (layer F.SilkS) (width 0.15))
+    (fp_line (start 8.15 6.55) (end 8.15 -6.55) (layer F.SilkS) (width 0.15))
+    (fp_line (start 8.15 -6.55) (end -8.15 -6.55) (layer F.SilkS) (width 0.15))
+    (fp_line (start -8.15 -6.55) (end -8.15 6.55) (layer F.SilkS) (width 0.15))
+    (pad GND smd rect (at -7.35 -5.85 90) (size 2 2) (layers F.Cu F.Paste F.Mask))
+    (pad GP5 smd rect (at 7.35 -5.85 90) (size 2 2) (layers F.Cu F.Paste F.Mask))
+    (pad GP16 smd rect (at -7.35 5.85 90) (size 2 2) (layers F.Cu F.Paste F.Mask))
+    (pad GP15 smd rect (at 7.35 5.85 90) (size 2 2) (layers F.Cu F.Paste F.Mask))
+    (pad GP14 smd rect (at -2.7 6.15 90) (size 1 1.2) (layers F.Cu F.Paste F.Mask))
+    (pad GP12 smd rect (at 0 6.15 90) (size 1 1.2) (layers F.Cu F.Paste F.Mask))
+    (pad GP13 smd rect (at 2.7 6.15 90) (size 1 1.2) (layers F.Cu F.Paste F.Mask))
+    (pad TX smd rect (at 0 -6.15 90) (size 1 1.2) (layers F.Cu F.Paste F.Mask))
+    (pad RST smd rect (at -2.7 -6.15 90) (size 1 1.2) (layers F.Cu F.Paste F.Mask))
+    (pad RX smd rect (at 2.7 -6.15 90) (size 1 1.2) (layers F.Cu F.Paste F.Mask))
+    (pad 3.3 smd rect (at -7.75 0 90) (size 1.2 1) (layers F.Cu F.Paste F.Mask))
+    (pad CHPD smd rect (at -7.75 2.9 90) (size 1.2 1) (layers F.Cu F.Paste F.Mask))
+    (pad ANT smd rect (at -7.75 -2.9 90) (size 1.2 1) (layers F.Cu F.Paste F.Mask))
+    (pad GP2 smd rect (at 7.75 0 90) (size 1.2 1) (layers F.Cu F.Paste F.Mask))
+    (pad GP0 smd rect (at 7.75 -2.9 90) (size 1.2 1) (layers F.Cu F.Paste F.Mask))
+    (pad GP4 smd rect (at 7.75 2.9 90) (size 1.2 1) (layers F.Cu F.Paste F.Mask))
+    (pad GND smd rect (at -1.3 -1.3 90) (size 2 2) (layers F.Cu F.Paste F.Mask))
+    (pad GND smd rect (at 1.3 -1.3 90) (size 2 2) (layers F.Cu F.Paste F.Mask))
+    (pad GND smd rect (at -1.3 1.3 90) (size 2 2) (layers F.Cu F.Paste F.Mask))
+    (pad GND smd rect (at 1.3 1.3 90) (size 2 2) (layers F.Cu F.Paste F.Mask))
+  )
   (gr_text D (at 142.24 80.518 90) (layer F.SilkS)

Commit message: 2016-sep
Parts:
- removed R1, R2, R3: R_0603, Resistors_SMD:R_0603
- added ?: Measurement_Point_Round-SMD-Pad_Small, Measurement_Points:Measurement_Point_Round-SMD-Pad_Small, F.Cu at (148.6, 73.0)
- added ?: Measurement_Point_Round-SMD-Pad_Small, Measurement_Points:Measurement_Point_Round-SMD-Pad_Small, F.Cu at (133.0, 72.4)
- moved ? 0.92 mm to (135.8, 41.7)
- moved WIFI ANT 0.18 mm to (151.1, 71.9)
Routing:
- net (no net): track 432.0 -> 429.1 mm, vias 12 -> 10
Other:
- board text added: "donp.org ESP-FTL 2016 Sep"
- board text removed: "donp.org ESP-FTL 2016 Aug"
