File: esp-ftl.kicad_pcb (KiCad board)
At the start: 2 copper layers, 21.3 x 43 mm, 16 parts

Commit message: random catchup
Parts:
- ? (x2): value MountingHole_2.2mm_M2 -> (none)
- ? (x2): value Measurement_Point_Round-SMD-Pad_Small -> (none)
Changed lines of the file:
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@@
-(kicad_pcb (version 4) (host pcbnew 4.1.0-alpha+201607031448+6962~45~ubuntu15.04.1-product)
+(kicad_pcb (version 4) (host pcbnew 4.0.4+e1-6308~48~ubuntu16.04.1-stable)
   (general
     (links 0)
     (no_connects 0)
-    (area 116.122572 34.4675 165.944429 88.983285)
+    (area 116.19757 34.45 165.36143 88.908287)
     (thickness 1.6)
     (drawings 20)
@@
       (hpglpenspeed 20)
       (hpglpendiameter 15)
+      (hpglpenoverlay 2)
       (psnegative false)
       (psa4output false)
@@
       (effects (font (size 1 1) (thickness 0.15)))
     )
-    (fp_text value MountingHole_2.2mm_M2 (at 0 3.2) (layer F.Fab)
+    (fp_text value "" (at 0 3.2) (layer F.Fab)
       (effects (font (size 1 1) (thickness 0.15)))
     )
@@
       (effects (font (size 1 1) (thickness 0.15)))
     )
-    (fp_text value MountingHole_2.2mm_M2 (at 0 3.2) (layer F.Fab)
+    (fp_text value "" (at 0 3.2) (layer F.Fab)
       (effects (font (size 1 1) (thickness 0.15)))
     )
@@
       (effects (font (size 1 1) (thickness 0.15)))
     )
-    (fp_text value Measurement_Point_Round-SMD-Pad_Small (at 0 2) (layer F.Fab)
+    (fp_text value "" (at 0 2) (layer F.Fab)
       (effects (font (size 1 1) (thickness 0.15)))
     )
@@
       (effects (font (size 1 1) (thickness 0.15)))
     )
-    (fp_text value Measurement_Point_Round-SMD-Pad_Small (at 0 2) (layer F.Fab)
-      (effects (font (size 1 1) (thickness 0.15)))
-    )
+    (fp_text value "" (at 0 2) (layer F.Fab)
+      (effects (font (size 1 1) (thickness 0.15)))
+    )
