File: neotiny.kicad_pcb (KiCad board)
At the start: 2 copper layers, 22 x 15.8 mm, 5 parts

Commit message: NeoTiny 2016 Dec
Parts:
- added ?: LED_1206, LEDs:LED_1206, F.Cu at (94.6, 84.1)
- added ?: R_0603, Resistors_SMD:R_0603, F.Cu at (89.8, 83.8)
- moved ? 7.91 mm to (99.9, 83.6), turned to 180 degrees
- moved ? 7.50 mm to (84.5, 72.4)
- moved ? 5.20 mm to (99.9, 71.9)
- moved 3535 1.94 mm to (94.7, 78.9)
- moved ATTINY 1.14 mm to (86.8, 78.6), turned to 90 degrees
Routing:
- net (no net): track 0.00 -> 133.4 mm, vias 0 -> 7
Other:
- board size 22 x 15.8 mm -> 21 x 15.8 mm
- board text added: "+ V"
- board text added: "+5.5"
- board text added: "+V"
- board text added: "1"
- board text added: "2.7v-5.5v"
- board text added: "3.7-5.5v"
- board text added: "D"
- board text added: "G N D"
- board text added: "IN"
- board text added: "NeoTiny 2016 Dec"
- board text added: "OUT"
- board text added: "donp.org"

Commit message: Jan 2017
Parts:
- added ?: R_0603, Resistors_SMD:R_0603, F.Cu at (94.9, 75.4)
- moved ? 0.66 mm to (83.8, 72.3)
Routing:
- net (no net): track 133.4 -> 130.6 mm
Other:
- board text added: "NeoTiny 2017 Jan"
- board text removed: "NeoTiny 2016 Dec"
Changed lines of the file:
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@@
     (thickness 1.6)
     (drawings 18)
-    (tracks 85)
+    (tracks 88)
     (zones 0)
-    (modules 7)
+    (modules 8)
     (nets 1)
   )
@@
     (uvia_drill 0.1)
   )
+  (module Resistors_SMD:R_0603 (layer F.Cu)
+    (at 94.9 75.4)
+    (descr "Resistor SMD 0603, reflow soldering, Vishay (see dcrcw.pdf)")
+    (tags "resistor 0603")
+    (attr smd)
+    (fp_text reference "" (at 0 -1.9) (layer F.SilkS)
+      (effects (font (size 1 1) (thickness 0.15)))
+    )
+    (fp_text value R_0603 (at 0 1.9) (layer F.Fab)
+      (effects (font (size 1 1) (thickness 0.15)))
+    )
+    (fp_line (start -0.8 0.4) (end -0.8 -0.4) (layer F.Fab) (width 0.1))
+    (fp_line (start 0.8 0.4) (end -0.8 0.4) (layer F.Fab) (width 0.1))
+    (fp_line (start 0.8 -0.4) (end 0.8 0.4) (layer F.Fab) (width 0.1))
+    (fp_line (start -0.8 -0.4) (end 0.8 -0.4) (layer F.Fab) (width 0.1))
+    (fp_line (start -1.3 -0.8) (end 1.3 -0.8) (layer F.CrtYd) (width 0.05))
+    (fp_line (start -1.3 0.8) (end 1.3 0.8) (layer F.CrtYd) (width 0.05))
+    (fp_line (start -1.3 -0.8) (end -1.3 0.8) (layer F.CrtYd) (width 0.05))
+    (fp_line (start 1.3 -0.8) (end 1.3 0.8) (layer F.CrtYd) (width 0.05))
+    (fp_line (start 0.5 0.675) (end -0.5 0.675) (layer F.SilkS) (width 0.15))
+    (fp_line (start -0.5 -0.675) (end 0.5 -0.675) (layer F.SilkS) (width 0.15))
+    (pad 1 smd rect (at -0.75 0) (size 0.5 0.9) (layers F.Cu F.Paste F.Mask))
+    (pad 2 smd rect (at 0.75 0) (size 0.5 0.9) (layers F.Cu F.Paste F.Mask))
+    (model Resistors_SMD.3dshapes/R_0603.wrl
+      (at (xyz 0 0 0))
+      (scale (xyz 1 1 1))
+      (rotate (xyz 0 0 0))
+    )
+  )
   (module Pin_Headers:Pin_Header_Straight_1x02 (layer F.Cu)
     (at 99.9 83.6 180)
@@
   )
   (module Pin_Headers:Pin_Header_Straight_1x04 (layer F.Cu)
-    (at 84.5 72.4 90)
+    (at 83.85 72.3 90)
     (descr "Through hole pin header")
     (tags "pin header")
@@
     (effects (font (size 0.9 0.9) (thickness 0.1)) (justify mirror))
   )
-  (gr_text "NeoTiny 2016 Dec" (at 86.6 85) (layer F.SilkS)
+  (gr_text "NeoTiny 2017 Jan" (at 86.6 85) (layer F.SilkS)
     (effects (font (size 0.8 0.8) (thickness 0.1)))
   )
@@
   (gr_line (start 81 69.8) (end 102 69.8) (angle 90) (layer Edge.Cuts) (width 0.15))
   (gr_line (start 81 69.8) (end 81 85.6) (angle 90) (layer Edge.Cuts) (width 0.15))
+  (segment (start 95.65 75.4) (end 96.6 75.4) (width 0.25) (layer F.Cu) (net 0))
+  (segment (start 97.56 74.44) (end 99.9 74.44) (width 0.25) (layer B.Cu) (net 0))
+  (segment (start 96.6 75.4) (end 97.56 74.44) (width 0.25) (layer B.Cu) (net 0))
+  (via (at 96.6 75.4) (size 0.6) (drill 0.4) (layers F.Cu B.Cu) (net 0))
+  (segment (start 93.95 75.2) (end 93.2 75.2) (width 0.25) (layer F.Cu) (net 0))
+  (segment (start 91.935 77.965) (end 89.975 77.965) (width 0.25) (layer F.Cu) (net 0))
+  (segment (start 91.935 77.965) (end 91.9 77.93) (width 0.25) (layer F.Cu) (net 0))
+  (segment (start 91.9 77.93) (end 91.9 76.4) (width 0.25) (layer F.Cu) (net 0))
+  (segment (start 91.9 76.4) (end 93.1 75.2) (width 0.25) (layer F.Cu) (net 0))
+  (segment (start 93.1 75.2) (end 93.2 75.2) (width 0.25) (layer F.Cu) (net 0))
+  (segment (start 93.95 75.2) (end 94.15 75.4) (width 0.25) (layer F.Cu) (net 0))
   (segment (start 96.3 81) (end 96.3 83.1) (width 0.25) (layer B.Cu) (net 0))
   (segment (start 97.3 84.1) (end 96.01986 84.1) (width 0.25) (layer F.Cu) (net 0))
@@
   (segment (start 91.2 76.8) (end 91.095 76.695) (width 0.25) (layer F.Cu) (net 0))
   (via (at 91.2 76.8) (size 0.6) (drill 0.4) (layers F.Cu B.Cu) (net 0))
-  (segment (start 89.975 77.965) (end 91.935 77.965) (width 0.25) (layer F.Cu) (net 0))
-  (segment (start 94.96 74.44) (end 99.9 74.44) (width 0.25) (layer B.Cu) (net 0))
-  (segment (start 94.8 74.6) (end 94.96 74.44) (width 0.25) (layer B.Cu) (net 0))
-  (via (at 94.8 74.6) (size 0.6) (drill 0.4) (layers F.Cu B.Cu) (net 0))
-  (segment (start 93.7 74.6) (end 94.8 74.6) (width 0.25) (layer F.Cu) (net 0))
-  (segment (start 91.9 76.4) (end 93.7 74.6) (width 0.25) (layer F.Cu) (net 0))
-  (segment (start 91.9 77.93) (end 91.9 76.4) (width 0.25) (layer F.Cu) (net 0))
-  (segment (start 91.935 77.965) (end 91.9 77.93) (width 0.25) (layer F.Cu) (net 0))
   (segment (start 97.8 78.9) (end 97.8 72.9) (width 0.25) (layer F.Cu) (net 0))
   (segment (start 98.8 71.9) (end 99.9 71.9) (width 0.25) (layer F.Cu) (net 0))
@@
   (segment (start 90.935 79.235) (end 91.2 79.5) (width 0.25) (layer F.Cu) (net 0))
   (segment (start 89.975 80.505) (end 89.975 81.425) (width 0.25) (layer F.Cu) (net 0))
-  (segment (start 92.12 74.28) (end 92.12 72.4) (width 0.25) (layer F.Cu) (net 0))
-  (segment (start 91 75.4) (end 92.12 74.28) (width 0.25) (layer F.Cu) (net 0))
-  (segment (start 88.4 75.4) (end 91 75.4) (width 0.25) (layer F.Cu) (net 0))
+  (segment (start 91.3 74.25) (end 91.47 72.3) (width 0.25) (layer F.Cu) (net 0) (status 800020))
+  (segment (start 90.95 75.25) (end 91.3 74.25) (width 0.25) (layer F.Cu) (net 0))
+  (segment (start 88.4 75.4) (end 90.95 75.25) (width 0.25) (layer F.Cu) (net 0))
   (via (at 88.4 75.4) (size 0.6) (drill 0.4) (layers F.Cu B.Cu) (net 0))
   (segment (start 88.4 81.8) (end 88.4 75.4) (width 0.25) (layer B.Cu) (net 0))
@@
   (segment (start 89.975 81.425) (end 89.6 81.8) (width 0.25) (layer F.Cu) (net 0))
   (segment (start 83.625 79.235) (end 82.035 79.235) (width 0.25) (layer F.Cu) (net 0))
-  (segment (start 81.5 75.4) (end 84.5 72.4) (width 0.25) (layer F.Cu) (net 0))
+  (segment (start 81.5 75.4) (end 83.85 72.3) (width 0.25) (layer F.Cu) (net 0) (status 20))
   (segment (start 81.5 78.7) (end 81.5 75.4) (width 0.25) (layer F.Cu) (net 0))
   (segment (start 82.035 79.235) (end 81.5 78.7) (width 0.25) (layer F.Cu) (net 0))
   (segment (start 83.625 77.965) (end 82.135 77.965) (width 0.25) (layer F.Cu) (net 0))
-  (segment (start 84.34 75.1) (end 87.04 72.4) (width 0.25) (layer F.Cu) (net 0))
+  (segment (start 84.34 75.1) (end 86.39 72.3) (width 0.25) (layer F.Cu) (net 0) (status 20))
   (segment (start 82.4 75.1) (end 84.34 75.1) (width 0.25) (layer F.Cu) (net 0))
   (segment (start 81.9 75.6) (end 82.4 75.1) (width 0.25) (layer F.Cu) (net 0))
@@
   (segment (start 82.135 77.965) (end 81.9 77.73) (width 0.25) (layer F.Cu) (net 0))
   (segment (start 83.625 76.695) (end 82.505 76.695) (width 0.25) (layer F.Cu) (net 0))
-  (segment (start 86.28 75.7) (end 89.58 72.4) (width 0.25) (layer F.Cu) (net 0))
+  (segment (start 86.28 75.7) (end 88.93 72.3) (width 0.25) (layer F.Cu) (net 0) (status 20))
   (segment (start 82.6 75.7) (end 86.28 75.7) (width 0.25) (layer F.Cu) (net 0))
   (segment (start 82.4 75.9) (end 82.6 75.7) (width 0.25) (layer F.Cu) (net 0))

Commit message: catchup
Other:
- board text added: "D a t a"
- board text removed: "D"
- board text removed: "IN"
- board text removed: "OUT"
Changed lines of the file:
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@@
-(kicad_pcb (version 4) (host pcbnew 4.0.4+e1-6308~48~ubuntu16.04.1-stable)
+(kicad_pcb (version 4) (host pcbnew 4.0.5-e0-6337~49~ubuntu16.04.1)
   (general
     (links 0)
     (no_connects 0)
-    (area 78.425 62.485713 109.814287 89.775)
+    (area 77.775 62.385713 109.814287 89.775)
     (thickness 1.6)
-    (drawings 18)
+    (drawings 15)
     (tracks 88)
     (zones 0)
@@
     (uvia_drill 0.1)
   )
+  (module Pin_Headers:Pin_Header_Straight_1x03 (layer F.Cu)
+    (at 99.9 71.9)
+    (descr "Through hole pin header")
+    (tags "pin header")
+    (fp_text reference "" (at 0 -5.1) (layer F.SilkS)
+      (effects (font (size 1 1) (thickness 0.15)))
+    )
+    (fp_text value Pin_Header_Straight_1x03 (at 0 -3.1) (layer F.Fab)
+      (effects (font (size 1 1) (thickness 0.15)))
+    )
+    (fp_line (start -1.75 -1.75) (end -1.75 6.85) (layer F.CrtYd) (width 0.05))
+    (fp_line (start 1.75 -1.75) (end 1.75 6.85) (layer F.CrtYd) (width 0.05))
+    (fp_line (start -1.75 -1.75) (end 1.75 -1.75) (layer F.CrtYd) (width 0.05))
+    (fp_line (start -1.75 6.85) (end 1.75 6.85) (layer F.CrtYd) (width 0.05))
+    (fp_line (start -1.27 1.27) (end -1.27 6.35) (layer F.SilkS) (width 0.15))
+    (fp_line (start -1.27 6.35) (end 1.27 6.35) (layer F.SilkS) (width 0.15))
+    (fp_line (start 1.27 6.35) (end 1.27 1.27) (layer F.SilkS) (width 0.15))
+    (fp_line (start 1.55 -1.55) (end 1.55 0) (layer F.SilkS) (width 0.15))
+    (fp_line (start 1.27 1.27) (end -1.27 1.27) (layer F.SilkS) (width 0.15))
+    (fp_line (start -1.55 0) (end -1.55 -1.55) (layer F.SilkS) (width 0.15))
+    (fp_line (start -1.55 -1.55) (end 1.55 -1.55) (layer F.SilkS) (width 0.15))
+    (pad 1 thru_hole rect (at 0 0) (size 2.032 1.7272) (drill 1.016) (layers *.Cu *.Mask))
+    (pad 2 thru_hole oval (at 0 2.54) (size 2.032 1.7272) (drill 1.016) (layers *.Cu *.Mask))
+    (pad 3 thru_hole oval (at 0 5.08) (size 2.032 1.7272) (drill 1.016) (layers *.Cu *.Mask))
+    (model Pin_Headers.3dshapes/Pin_Header_Straight_1x03.wrl
+      (at (xyz 0 -0.1 0))
+      (scale (xyz 1 1 1))
+      (rotate (xyz 0 0 90))
+    )
+  )
   (module Resistors_SMD:R_0603 (layer F.Cu)
     (at 94.9 75.4)
@@
     )
   )
-  (module ws2812:3535 (layer F.Cu)
-    (at 94.7 78.9)
-    (fp_text reference 3535 (at 0 2.4) (layer F.SilkS)
-      (effects (font (size 0.9 0.9) (thickness 0.1)))
-    )
-    (fp_text value 3535 (at 0.05 -2.2) (layer F.Fab)
-      (effects (font (size 1 1) (thickness 0.15)))
-    )
-    (fp_line (start 1.75 1.75) (end -1.75 1.75) (layer F.SilkS) (width 0.15))
-    (fp_line (start -1.75 1.75) (end -1.75 -1.75) (layer F.SilkS) (width 0.15))
-    (fp_line (start 1.75 -1.75) (end 1.75 1.75) (layer F.SilkS) (width 0.15))
-    (fp_line (start -1.75 -1.75) (end 1.7 -1.75) (layer F.SilkS) (width 0.15))
-    (pad IN smd rect (at 1.325 0.875) (size 1.05 0.85) (drill (offset 0.1 0)) (layers F.Cu F.Paste F.Mask))
-    (pad VDD smd rect (at 1.325 -0.875) (size 1.05 0.85) (drill (offset 0.1 0)) (layers F.Cu F.Paste F.Mask))
-    (pad GND smd rect (at -1.325 0.875) (size 1.05 0.85) (drill (offset -0.1 0)) (layers F.Cu F.Paste F.Mask))
-    (pad OUT smd rect (at -1.325 -0.875) (size 1.05 0.85) (drill (offset -0.1 0)) (layers F.Cu F.Paste F.Mask))
-  )
   (module Pin_Headers:Pin_Header_Straight_1x04 (layer F.Cu)
     (at 83.85 72.3 90)
@@
     (model Pin_Headers.3dshapes/Pin_Header_Straight_1x04.wrl
       (at (xyz 0 -0.15 0))
-      (scale (xyz 1 1 1))
-      (rotate (xyz 0 0 90))
-    )
-  )
-  (module Pin_Headers:Pin_Header_Straight_1x03 (layer F.Cu)
-    (at 99.9 71.9)
-    (descr "Through hole pin header")
-    (tags "pin header")
-    (fp_text reference "" (at 0 -5.1) (layer F.SilkS)
-      (effects (font (size 1 1) (thickness 0.15)))
-    )
-    (fp_text value Pin_Header_Straight_1x03 (at 0 -3.1) (layer F.Fab)
-      (effects (font (size 1 1) (thickness 0.15)))
-    )
-    (fp_line (start -1.75 -1.75) (end -1.75 6.85) (layer F.CrtYd) (width 0.05))
-    (fp_line (start 1.75 -1.75) (end 1.75 6.85) (layer F.CrtYd) (width 0.05))
-    (fp_line (start -1.75 -1.75) (end 1.75 -1.75) (layer F.CrtYd) (width 0.05))
-    (fp_line (start -1.75 6.85) (end 1.75 6.85) (layer F.CrtYd) (width 0.05))
-    (fp_line (start -1.27 1.27) (end -1.27 6.35) (layer F.SilkS) (width 0.15))
-    (fp_line (start -1.27 6.35) (end 1.27 6.35) (layer F.SilkS) (width 0.15))
-    (fp_line (start 1.27 6.35) (end 1.27 1.27) (layer F.SilkS) (width 0.15))
-    (fp_line (start 1.55 -1.55) (end 1.55 0) (layer F.SilkS) (width 0.15))
-    (fp_line (start 1.27 1.27) (end -1.27 1.27) (layer F.SilkS) (width 0.15))
-    (fp_line (start -1.55 0) (end -1.55 -1.55) (layer F.SilkS) (width 0.15))
-    (fp_line (start -1.55 -1.55) (end 1.55 -1.55) (layer F.SilkS) (width 0.15))
-    (pad 1 thru_hole rect (at 0 0) (size 2.032 1.7272) (drill 1.016) (layers *.Cu *.Mask))
-    (pad 2 thru_hole oval (at 0 2.54) (size 2.032 1.7272) (drill 1.016) (layers *.Cu *.Mask))
-    (pad 3 thru_hole oval (at 0 5.08) (size 2.032 1.7272) (drill 1.016) (layers *.Cu *.Mask))
-    (model Pin_Headers.3dshapes/Pin_Header_Straight_1x03.wrl
-      (at (xyz 0 -0.1 0))
       (scale (xyz 1 1 1))
       (rotate (xyz 0 0 90))
@@
     )
   )
-  (gr_text D (at 101.6 74.5) (layer F.SilkS)
-    (effects (font (size 0.9 0.9) (thickness 0.1)))
-  )
-  (gr_text OUT (at 94.5 78.1) (layer F.SilkS)
-    (effects (font (size 0.3 0.3) (thickness 0.05)))
-  )
-  (gr_text IN (at 95.2 79.8) (layer F.SilkS)
-    (effects (font (size 0.3 0.3) (thickness 0.05)))
+  (module ws2812:3535 (layer F.Cu)
+    (at 94.7 78.9)
+    (fp_text reference 3535 (at 0 2.4) (layer F.SilkS)
+      (effects (font (size 0.9 0.9) (thickness 0.1)))
+    )
+    (fp_text value 3535 (at 0.05 -2.2) (layer F.Fab)
+      (effects (font (size 1 1) (thickness 0.15)))
+    )
+    (fp_line (start -0.4 0.7) (end 0.4 0.7) (layer F.SilkS) (width 0.15))
+    (fp_line (start 0.4 0.7) (end 0.4 1.1) (layer F.SilkS) (width 0.15))
+    (fp_line (start 0.4 1.1) (end -0.4 1.1) (layer F.SilkS) (width 0.15))
+    (fp_line (start -0.4 1.1) (end -0.4 0.7) (layer F.SilkS) (width 0.15))
+    (fp_line (start 1.75 1.75) (end -1.75 1.75) (layer F.SilkS) (width 0.15))
+    (fp_line (start -1.75 1.75) (end -1.75 -1.75) (layer F.SilkS) (width 0.15))
+    (fp_line (start 1.75 -1.75) (end 1.75 1.75) (layer F.SilkS) (width 0.15))
+    (fp_line (start -1.75 -1.75) (end 1.7 -1.75) (layer F.SilkS) (width 0.15))
+    (pad IN smd rect (at 1.325 0.875) (size 1.05 0.85) (drill (offset 0.1 0)) (layers F.Cu F.Paste F.Mask))
+    (pad VDD smd rect (at 1.325 -0.875) (size 1.05 0.85) (drill (offset 0.1 0)) (layers F.Cu F.Paste F.Mask))
+    (pad GND smd rect (at -1.325 0.875) (size 1.05 0.85) (drill (offset -0.1 0)) (layers F.Cu F.Paste F.Mask))
+    (pad OUT smd rect (at -1.325 -0.875) (size 1.05 0.85) (drill (offset -0.1 0)) (layers F.Cu F.Paste F.Mask))
+  )
+  (gr_text "D\na\nt\na\n" (at 101.45 74.5) (layer F.SilkS)
+    (effects (font (size 0.3 0.5) (thickness 0.03)))
   )
   (gr_text "+\nV" (at 95.3 78.1) (layer F.SilkS)
-    (effects (font (size 0.3 0.3) (thickness 0.05)))
-  )
-  (gr_text "G\nN\nD" (at 94.2 79.6) (layer F.SilkS)
     (effects (font (size 0.3 0.3) (thickness 0.05)))
   )
@@
   (segment (start 90.935 79.235) (end 91.2 79.5) (width 0.25) (layer F.Cu) (net 0))
   (segment (start 89.975 80.505) (end 89.975 81.425) (width 0.25) (layer F.Cu) (net 0))
-  (segment (start 91.3 74.25) (end 91.47 72.3) (width 0.25) (layer F.Cu) (net 0) (status 800020))
+  (segment (start 91.3 74.25) (end 91.47 72.3) (width 0.25) (layer F.Cu) (net 0) (status 20))
   (segment (start 90.95 75.25) (end 91.3 74.25) (width 0.25) (layer F.Cu) (net 0))
   (segment (start 88.4 75.4) (end 90.95 75.25) (width 0.25) (layer F.Cu) (net 0))
