File: neotiny.kicad_pcb (KiCad board)
At the start: 2 copper layers, 21 x 15.8 mm, 8 parts

Commit message: neotiny 2019
Parts:
- removed the ? at (94.9, 75.4)
- added REF**: MountingHole_1.2mm_M2, neotiny:MountingHole_1.2mm_M2, F.Cu at (95.8, 72.0)
- added REF**: MountingHole_1.2mm_M2, neotiny:MountingHole_1.2mm_M2, F.Cu at (83.0, 83.7)
Other:
- board text added: "NeoTiny 2019 Jan"
- board text added: "PB0"
- board text added: "PB1"
- board text added: "PB2"
- board text added: "PB5"
- board text removed: "NeoTiny 2017 Jan"
