File: esp-square.kicad_pcb (KiCad board)
At the start: 2 copper layers, 21.3 x 27.8 mm, 14 parts

Commit message: square rev-c fixes
Parts:
- added 3535: 3535, ws2812:3535, F.Cu at (146.1, 58.4)
- moved 3535 2.54 mm to (140.2, 58.4)
- moved ESP-06 0.51 mm to (142.5, 52.6)
Routing:
- net (no net): track 194.0 -> 205.7 mm, vias 6 -> 8

Commit message: PIN 9 IS ALWAYS GROUNDED
Parts:
- added ?: VEML6040, veml-rgb:VEML6040, F.Cu at (151.6, 58.4)
Routing:
- net (no net): track 205.7 -> 240.5 mm, vias 8 -> 12
Other:
- board text added: "1 GND"
- board text added: "4 +v"
- board text added: "donp.org 2017 May"
- board text added: "esp-square rev E1"
- board text removed: "donp.org 2016 Sep"
- board text removed: "esp-square rev C"
Changed lines of the file:
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@@
-(kicad_pcb (version 4) (host pcbnew 4.1.0-alpha+201607031448+6962~45~ubuntu15.04.1-product)
+(kicad_pcb (version 4) (host pcbnew 4.0.5-e0-6337~49~ubuntu16.04.1)
   (general
     (links 0)
     (no_connects 0)
-    (area 123.678215 35.86461 161.627286 73.743285)
+    (area 123.753213 35.8481 161.552287 73.668287)
     (thickness 1.6)
-    (drawings 7)
-    (tracks 116)
+    (drawings 9)
+    (tracks 153)
     (zones 0)
-    (modules 15)
+    (modules 16)
     (nets 1)
   )
@@
     (mod_text_size 1 1)
     (mod_text_width 0.15)
-    (pad_size 0.39878 1.3462)
+    (pad_size 0.45 0.35)
     (pad_drill 0)
     (pad_to_mask_clearance 0.2)
@@
       (hpglpenspeed 20)
       (hpglpendiameter 15)
+      (hpglpenoverlay 2)
       (psnegative false)
       (psa4output false)
@@
     (pad 1 np_thru_hole circle (at 0 0) (size 2.2 2.2) (drill 2.2) (layers *.Cu *.Mask F.SilkS))
   )
+  (module veml-rgb:VEML6040 (layer F.Cu)
+    (at 151.6126 58.42)
+    (fp_text reference "" (at 0.24 2.46) (layer F.SilkS)
+      (effects (font (size 1 1) (thickness 0.15)))
+    )
+    (fp_text value VEML6040 (at 0 -0.5) (layer F.Fab)
+      (effects (font (size 1 1) (thickness 0.15)))
+    )
+    (fp_line (start -1.2 0.5) (end -1.2 1.65) (layer F.SilkS) (width 0.06))
+    (fp_line (start -1.2 1.65) (end 0.86 1.65) (layer F.SilkS) (width 0.1))
+    (fp_line (start 0.86 1.65) (end 0.86 0.5) (layer F.SilkS) (width 0.06))
+    (fp_line (start -1.2 0.5) (end 0.86 0.5) (layer F.SilkS) (width 0.1))
+    (pad GND smd rect (at -0.945 0.725) (size 0.45 0.35) (layers F.Cu F.Paste F.Mask))
+    (pad +V smd rect (at 0.605 0.725) (size 0.45 0.35) (layers F.Cu F.Paste F.Mask))
+    (pad 3 smd rect (at 0.605 1.425) (size 0.45 0.35) (layers F.Cu F.Paste F.Mask))
+    (pad 4 smd rect (at -0.895 1.425) (size 0.55 0.35) (layers F.Cu F.Paste F.Mask))
+  )
+  (gr_text "1\nGND" (at 149.9616 59.0804) (layer F.SilkS)
+    (effects (font (size 0.2 0.2) (thickness 0.05)))
+  )
+  (gr_text "4\n+v" (at 152.8826 59.1312) (layer F.SilkS)
+    (effects (font (size 0.2 0.2) (thickness 0.05)))
+  )
   (gr_text "|_|0|_|\n|_|_|0|\n|0|0|0|" (at 150.876 40.767) (layer B.SilkS)
     (effects (font (size 0.7 0.7) (thickness 0.1)))
   )
-  (gr_text "esp-square\nrev C" (at 151.892 55.626 90) (layer F.SilkS)
+  (gr_text "esp-square\nrev E1" (at 151.892 55.626 90) (layer F.SilkS)
     (effects (font (size 0.7 0.7) (thickness 0.1)))
   )
@@
   (gr_line (start 132 65.76) (end 153.3 65.76) (angle 90) (layer Edge.Cuts) (width 0.2))
   (gr_line (start 153.3 38) (end 132 38) (angle 90) (layer Edge.Cuts) (width 0.2))
-  (gr_text "donp.org\n2016 Sep" (at 150.749 42.418) (layer F.SilkS)
+  (gr_text "donp.org\n2017 May" (at 150.749 42.418) (layer F.SilkS)
     (effects (font (size 0.6 0.6) (thickness 0.1)))
   )
-  (segment (start 142.6845 63.754) (end 142.6845 62.1665) (width 0.25) (layer B.Cu) (net 0) (status 400000))
-  (segment (start 141.194 61.692) (end 141.194 53.878) (width 0.25) (layer B.Cu) (net 0) (status 800000))
+  (segment (start 148.59 57.658) (end 148.59 59.682) (width 0.25) (layer B.Cu) (net 0) (status 800000))
+  (segment (start 148.59 59.682) (end 148.344 59.928) (width 0.25) (layer B.Cu) (net 0) (status C00000))
+  (segment (start 148.344 59.928) (end 149.209 59.928) (width 0.25) (layer B.Cu) (net 0))
+  (segment (start 149.209 59.928) (end 150.0124 60.7314) (width 0.25) (layer B.Cu) (net 0))
+  (segment (start 150.7176 60.7) (end 150.7176 59.845) (width 0.25) (layer F.Cu) (net 0))
+  (segment (start 150.749 60.7314) (end 150.7176 60.7) (width 0.25) (layer F.Cu) (net 0))
+  (via (at 150.749 60.7314) (size 0.6) (drill 0.4) (layers F.Cu B.Cu) (net 0))
+  (segment (start 150.0124 60.7314) (end 150.749 60.7314) (width 0.25) (layer B.Cu) (net 0))
+  (segment (start 145.394 60.328) (end 145.394 61.3454) (width 0.25) (layer B.Cu) (net 0))
+  (segment (start 152.2176 60.7268) (end 152.2176 59.845) (width 0.25) (layer F.Cu) (net 0))
+  (segment (start 152.2222 60.7314) (end 152.2176 60.7268) (width 0.25) (layer F.Cu) (net 0))
+  (via (at 152.2222 60.7314) (size 0.6) (drill 0.4) (layers F.Cu B.Cu) (net 0))
+  (segment (start 152.2222 61.2902) (end 152.2222 60.7314) (width 0.25) (layer B.Cu) (net 0))
+  (segment (start 152.3238 61.3918) (end 152.2222 61.2902) (width 0.25) (layer B.Cu) (net 0))
+  (segment (start 150.622 61.3918) (end 152.3238 61.3918) (width 0.25) (layer B.Cu) (net 0))
+  (segment (start 150.4188 61.595) (end 150.622 61.3918) (width 0.25) (layer B.Cu) (net 0))
+  (segment (start 145.6436 61.595) (end 150.4188 61.595) (width 0.25) (layer B.Cu) (net 0))
+  (segment (start 145.394 61.3454) (end 145.6436 61.595) (width 0.25) (layer B.Cu) (net 0))
+  (segment (start 150.6676 59.145) (end 150.6676 58.2878) (width 0.25) (layer F.Cu) (net 0))
+  (segment (start 150.0378 57.658) (end 148.59 57.658) (width 0.25) (layer F.Cu) (net 0))
+  (segment (start 150.6676 58.2878) (end 150.0378 57.658) (width 0.25) (layer F.Cu) (net 0))
+  (segment (start 152.1968 58.1152) (end 152.1968 59.1242) (width 0.25) (layer F.Cu) (net 0))
+  (segment (start 152.1968 59.1242) (end 152.2176 59.145) (width 0.25) (layer F.Cu) (net 0))
+  (segment (start 148.97037 45.881646) (end 148.97037 46.58297) (width 0.25) (layer F.Cu) (net 0))
+  (segment (start 152.1968 53.6448) (end 152.1968 58.1152) (width 0.25) (layer F.Cu) (net 0))
+  (segment (start 152.1968 58.1152) (end 152.1968 58.1914) (width 0.25) (layer F.Cu) (net 0))
+  (segment (start 151.5618 53.0098) (end 152.1968 53.6448) (width 0.25) (layer F.Cu) (net 0))
+  (segment (start 150.6474 53.0098) (end 151.5618 53.0098) (width 0.25) (layer F.Cu) (net 0))
+  (segment (start 149.86 52.2224) (end 150.6474 53.0098) (width 0.25) (layer F.Cu) (net 0))
+  (segment (start 149.86 49.8856) (end 149.86 52.2224) (width 0.25) (layer F.Cu) (net 0))
+  (segment (start 148.5138 48.5394) (end 149.86 49.8856) (width 0.25) (layer F.Cu) (net 0))
+  (via (at 148.5138 48.5394) (size 0.6) (drill 0.4) (layers F.Cu B.Cu) (net 0))
+  (segment (start 148.5138 47.7012) (end 148.5138 48.5394) (width 0.25) (layer B.Cu) (net 0))
+  (segment (start 149.3012 46.9138) (end 148.5138 47.7012) (width 0.25) (layer B.Cu) (net 0))
+  (via (at 149.3012 46.9138) (size 0.6) (drill 0.4) (layers F.Cu B.Cu) (net 0))
+  (segment (start 148.97037 46.58297) (end 149.3012 46.9138) (width 0.25) (layer F.Cu) (net 0))
+  (segment (start 142.6845 63.754) (end 142.6845 62.1665) (width 0.25) (layer B.Cu) (net 0))
+  (segment (start 141.194 61.692) (end 141.194 53.878) (width 0.25) (layer B.Cu) (net 0))
   (segment (start 141.224 61.722) (end 141.194 61.692) (width 0.25) (layer B.Cu) (net 0))
   (segment (start 142.24 61.722) (end 141.224 61.722) (width 0.25) (layer B.Cu) (net 0))
   (segment (start 142.6845 62.1665) (end 142.24 61.722) (width 0.25) (layer B.Cu) (net 0))
-  (segment (start 142.494 60.328) (end 142.878 60.328) (width 0.25) (layer B.Cu) (net 0) (status C00000))
-  (segment (start 142.878 60.328) (end 145.2245 62.6745) (width 0.25) (layer B.Cu) (net 0) (status 400000))
-  (segment (start 145.2245 62.6745) (end 145.2245 63.754) (width 0.25) (layer B.Cu) (net 0) (status 800000))
-  (segment (start 147.375 57.545) (end 148.477 57.545) (width 0.25) (layer F.Cu) (net 0) (status 400000))
+  (segment (start 142.494 60.328) (end 142.878 60.328) (width 0.25) (layer B.Cu) (net 0))
+  (segment (start 142.878 60.328) (end 145.2245 62.6745) (width 0.25) (layer B.Cu) (net 0))
+  (segment (start 145.2245 62.6745) (end 145.2245 63.754) (width 0.25) (layer B.Cu) (net 0))
+  (segment (start 147.375 57.545) (end 148.477 57.545) (width 0.25) (layer F.Cu) (net 0))
   (segment (start 148.59 57.658) (end 146.558 57.658) (width 0.25) (layer B.Cu) (net 0))
   (via (at 148.59 57.658) (size 0.6) (drill 0.4) (layers F.Cu B.Cu) (net 0))
   (segment (start 148.477 57.545) (end 148.59 57.658) (width 0.25) (layer F.Cu) (net 0))
-  (segment (start 141.533 57.545) (end 142.099 57.545) (width 0.25) (layer F.Cu) (net 0) (status C00000))
-  (segment (start 142.099 57.545) (end 142.748 56.896) (width 0.25) (layer F.Cu) (net 0) (status 400000))
+  (segment (start 141.533 57.545) (end 142.099 57.545) (width 0.25) (layer F.Cu) (net 0))
+  (segment (start 142.099 57.545) (end 142.748 56.896) (width 0.25) (layer F.Cu) (net 0))
   (via (at 142.748 56.896) (size 0.6) (drill 0.4) (layers F.Cu B.Cu) (net 0))
   (segment (start 142.748 56.896) (end 143.794 55.85) (width 0.25) (layer B.Cu) (net 0))
-  (segment (start 143.794 55.85) (end 143.794 53.878) (width 0.25) (layer B.Cu) (net 0) (status 800000))
+  (segment (start 143.794 55.85) (end 143.794 53.878) (width 0.25) (layer B.Cu) (net 0))
   (segment (start 133.6675 47.752) (end 140.38834 47.752) (width 0.25) (layer F.Cu) (net 0))
   (segment (start 140.38834 47.752) (end 140.56614 47.5742) (width 0.25) (layer F.Cu) (net 0))
@@
   (segment (start 148.644 49.878) (end 150.462 49.37) (width 0.25) (layer B.Cu) (net 0) (status 10))
   (segment (start 150.462 49.37) (end 151.638 50.546) (width 0.25) (layer B.Cu) (net 0))
-  (segment (start 142.875 45.974) (end 151.257 45.847) (width 0.25) (layer F.Cu) (net 0))
+  (segment (start 142.875 45.974) (end 148.97037 45.881646) (width 0.25) (layer F.Cu) (net 0))
+  (segment (start 148.97037 45.881646) (end 151.257 45.847) (width 0.25) (layer F.Cu) (net 0))
   (segment (start 151.257 45.847) (end 151.638 45.466) (width 0.25) (layer F.Cu) (net 0))
   (segment (start 146.558 46.99) (end 148.082 46.99) (width 0.25) (layer F.Cu) (net 0))

Commit message: rev E1
Parts:
- removed the 3535 at (146.1, 58.4)
- moved ? 5.91 mm to (145.9, 56.7)
Routing:
- net (no net): track 240.5 -> 212.6 mm, vias 12 -> 9
Other:
- board text added: "+3.3"
- board text added: "+4-12v"
- board text added: "+V"
- board text added: "4 +3.3v"
- board text added: "GND"
- board text added: "IO0"
- board text added: "IO14"
- board text added: "IO2"
- board text added: "RX"
- board text added: "SCL 3"
- board text added: "SDA 2"
- board text added: "TX"
- board text removed: "4 +v"

Commit message: rev D1 (SPI)
Parts:
- added ?: R_0603, Resistors_SMD:R_0603, F.Cu at (147.8, 60.5)
- ?: footprint Pin_Headers:Pin_Header_Straight_1x03 -> Pin_Headers:Pin_Header_Straight_1x06_Pitch2.54mm
Routing:
- net (no net): track 212.6 -> 223.9 mm, vias 9 -> 10
Other:
- board text added: "I12"
- board text added: "I13"
- board text added: "I14"
- board text added: "I15"
- board text added: "rev D1"
- board text removed: "IO14"
- board text removed: "esp-square rev E1"
