File: breakouts/qfn32.kicad_pcb (KiCad board)
At the start: 2 copper layers, 21.2 x 44 mm, 6 parts

Commit message: catchup
Parts:
- removed 10pf (x2): C_0603_HandSoldering, Capacitors_SMD:C_0603_HandSoldering
- removed 26mhz: Crystal_SMD_2016-4pin_2.0x1.6mm, Crystals:Crystal_SMD_2016-4pin_2.0x1.6mm
- removed QFN-32 0.5mm: QFN-32-1EP_5x5mm_Pitch0.5mm, Housings_DFN_QFN:QFN-32-1EP_5x5mm_Pitch0.5mm
- added QFN-32 0.4mm: QFN-32-1EP_4x4mm_Pitch0.4mm, Housings_DFN_QFN:QFN-32-1EP_4x4mm_Pitch0.4mm, F.Cu at (135.9, 76.2)
Routing:
- net (no net): track 505.1 -> 0.00 mm, vias 4 -> 0
Other:
- board text removed: "8285 +clk"
- board text removed: "donp.org"
