File: breakouts/micamp.kicad_pcb (KiCad board)
At the start: 2 copper layers, 16.2 x 8.5 mm, 4 parts

Commit message: micamp catchup
Parts:
- ? (x2): value Pin_Header_Straight_1x02_Pitch2.54mm -> (none)
Changed lines of the file:
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@@
       (effects (font (size 1 1) (thickness 0.15)))
     )
-    (fp_text value Pin_Header_Straight_1x02_Pitch2.54mm (at 0 7.47) (layer F.Fab)
+    (fp_text value "" (at 0 7.47) (layer F.Fab)
       (effects (font (size 1 1) (thickness 0.15)))
     )
@@
       (effects (font (size 1 1) (thickness 0.15)))
     )
-    (fp_text value Pin_Header_Straight_1x02_Pitch2.54mm (at 0 7.47) (layer F.Fab)
+    (fp_text value "" (at 0 7.47) (layer F.Fab)
       (effects (font (size 1 1) (thickness 0.15)))
     )
@@
   (gr_line (start 125.254 65.2058) (end 141.4526 65.2058) (angle 90) (layer Edge.Cuts) (width 0.2))
   (gr_line (start 125.254 56.7018) (end 141.4526 56.7018) (angle 90) (layer Edge.Cuts) (width 0.2))
-  (segment (start 136.586 59.687) (end 137.3602 59.687) (width 0.25) (layer F.Cu) (net 0) (status 400000))
-  (segment (start 137.922 60.96) (end 139.7 60.96) (width 0.25) (layer F.Cu) (net 0) (status 800000))
+  (segment (start 136.586 59.687) (end 137.3602 59.687) (width 0.25) (layer F.Cu) (net 0))
+  (segment (start 137.922 60.96) (end 139.7 60.96) (width 0.25) (layer F.Cu) (net 0))
   (segment (start 137.668 60.706) (end 137.922 60.96) (width 0.25) (layer F.Cu) (net 0))
   (segment (start 137.668 59.9948) (end 137.668 60.706) (width 0.25) (layer F.Cu) (net 0))
   (segment (start 137.3602 59.687) (end 137.668 59.9948) (width 0.25) (layer F.Cu) (net 0))
-  (segment (start 136.586 62.487) (end 136.586 62.672) (width 0.25) (layer F.Cu) (net 0) (status C00000))
-  (segment (start 136.586 62.672) (end 137.414 63.5) (width 0.25) (layer F.Cu) (net 0) (status 400000))
-  (segment (start 137.414 63.5) (end 139.7 63.5) (width 0.25) (layer F.Cu) (net 0) (status 800000))
-  (segment (start 134.686 62.487) (end 133.601 62.487) (width 0.25) (layer F.Cu) (net 0) (status 400000))
-  (segment (start 129.4892 58.42) (end 127 58.42) (width 0.25) (layer B.Cu) (net 0) (status 800000))
+  (segment (start 136.586 62.487) (end 136.586 62.672) (width 0.25) (layer F.Cu) (net 0))
+  (segment (start 136.586 62.672) (end 137.414 63.5) (width 0.25) (layer F.Cu) (net 0))
+  (segment (start 137.414 63.5) (end 139.7 63.5) (width 0.25) (layer F.Cu) (net 0))
+  (segment (start 134.686 62.487) (end 133.601 62.487) (width 0.25) (layer F.Cu) (net 0))
+  (segment (start 129.4892 58.42) (end 127 58.42) (width 0.25) (layer B.Cu) (net 0))
   (segment (start 133.5786 62.5094) (end 129.4892 58.42) (width 0.25) (layer B.Cu) (net 0))
   (via (at 133.5786 62.5094) (size 0.6) (drill 0.4) (layers F.Cu B.Cu) (net 0))
   (segment (start 133.601 62.487) (end 133.5786 62.5094) (width 0.25) (layer F.Cu) (net 0))
   (segment (start 134.7216 58.42) (end 132.08 58.42) (width 0.25) (layer F.Cu) (net 0))
-  (segment (start 131.973 58.527) (end 131.973 60.1704) (width 0.25) (layer F.Cu) (net 0) (status 800000))
+  (segment (start 131.973 58.527) (end 131.973 60.1704) (width 0.25) (layer F.Cu) (net 0))
   (segment (start 132.08 58.42) (end 131.973 58.527) (width 0.25) (layer F.Cu) (net 0))
-  (segment (start 139.7 58.42) (end 134.7216 58.42) (width 0.25) (layer F.Cu) (net 0) (status 400000))
+  (segment (start 139.7 58.42) (end 134.7216 58.42) (width 0.25) (layer F.Cu) (net 0))
   (segment (start 134.7216 58.42) (end 134.6708 58.42) (width 0.25) (layer F.Cu) (net 0))
-  (segment (start 134.686 58.4352) (end 134.686 59.687) (width 0.25) (layer F.Cu) (net 0) (status 800000))
+  (segment (start 134.686 58.4352) (end 134.686 59.687) (width 0.25) (layer F.Cu) (net 0))
   (segment (start 134.6708 58.42) (end 134.686 58.4352) (width 0.25) (layer F.Cu) (net 0))
   (segment (start 132.0038 63.5) (end 133.1214 63.5) (width 0.25) (layer F.Cu) (net 0))
-  (segment (start 135.636 64.643) (end 135.636 62.487) (width 0.25) (layer F.Cu) (net 0) (status 800000))
+  (segment (start 135.636 64.643) (end 135.636 62.487) (width 0.25) (layer F.Cu) (net 0))
   (segment (start 133.1722 64.643) (end 135.636 64.643) (width 0.25) (layer F.Cu) (net 0))
   (segment (start 133.1214 64.5922) (end 133.1722 64.643) (width 0.25) (layer F.Cu) (net 0))
