File: pcb/breakouts/8285.kicad_pcb (KiCad board)
At the start: 2 copper layers, 21.2 x 41.5 mm, 6 parts

Commit message: connect crystal to pinout
Parts:
- 10pf: value C_0603_HandSoldering -> (none)
Routing:
- net (no net): track 483.6 -> 504.6 mm, vias 3 -> 5
Other:
- board text added: "2019-Mar-8"
Changed lines of the file:
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@@
-(kicad_pcb (version 4) (host pcbnew 4.0.5-e0-6337~49~ubuntu16.04.1)
+(kicad_pcb (version 20171130) (host pcbnew 5.0.2-bee76a0~70~ubuntu18.04.1)
   (general
-    (links 0)
-    (no_connects 0)
-    (area 111.799999 52.515 159.980001 99.985)
     (thickness 1.6)
-    (drawings 11)
-    (tracks 136)
+    (drawings 12)
+    (tracks 157)
     (zones 0)
     (modules 6)
@@
     (pad_drill 1)
     (pad_to_mask_clearance 0.2)
+    (solder_mask_min_width 0.25)
     (aux_axis_origin 0 0)
     (visible_elements FFFEFFFF)
@@
       (layerselection 0x010f0_80000001)
       (usegerberextensions true)
+      (usegerberattributes false)
+      (usegerberadvancedattributes false)
+      (creategerberjobfile false)
       (excludeedgelayer true)
       (linewidth 0.100000)
@@
       (hpglpennumber 1)
       (hpglpenspeed 20)
-      (hpglpendiameter 15)
-      (hpglpenoverlay 2)
+      (hpglpendiameter 15.000000)
       (psnegative false)
       (psa4output false)
@@
       (drillshape 0)
       (scaleselection 1)
-      (outputdirectory /home/donp/osh))
+      (outputdirectory "/home/donp/osh"))
   )
   (net 0 "")
@@
       (effects (font (size 1 1) (thickness 0.15)))
     )
-    (fp_text value C_0603_HandSoldering (at 0 1.5) (layer F.Fab)
+    (fp_text value "" (at 0 1.5) (layer F.Fab) hide
       (effects (font (size 1 1) (thickness 0.15)))
     )
@@
     (tags "SMD SMT crystal")
     (attr smd)
-    (fp_text reference 26mhz (at -0.0254 -1.7526) (layer F.SilkS)
+    (fp_text reference 26mhz (at -0.0254 -1.7526) (layer F.SilkS) hide
       (effects (font (size 1 1) (thickness 0.15)))
     )
@@
       (effects (font (size 1 1) (thickness 0.15)))
     )
-    (fp_text value Pin_Header_Straight_1x08_Pitch2.54mm (at 0 40.49) (layer F.Fab)
+    (fp_text value Pin_Header_Straight_1x08_Pitch2.54mm (at 0 40.49) (layer F.Fab) hide
       (effects (font (size 1 1) (thickness 0.15)))
     )
@@
     (pad 16 thru_hole oval (at 0 38.1) (size 1.7 1.7) (drill 1) (layers *.Cu *.Mask))
     (model Pin_Headers.3dshapes/Pin_Header_Straight_1x16_Pitch2.54mm.wrl
-      (at (xyz 0 -0.75 0))
+      (offset (xyz 0 -19.04999971389771 0))
       (scale (xyz 1 1 1))
       (rotate (xyz 0 0 90))
@@
     (pad 16 thru_hole oval (at 0 38.1) (size 1.7 1.7) (drill 1) (layers *.Cu *.Mask))
     (model Pin_Headers.3dshapes/Pin_Header_Straight_1x16_Pitch2.54mm.wrl
-      (at (xyz 0 -0.75 0))
+      (offset (xyz 0 -19.04999971389771 0))
       (scale (xyz 1 1 1))
       (rotate (xyz 0 0 90))
     )
+  )
+  (gr_text 2019-Mar-8 (at 135.9662 94.234) (layer F.SilkS)
+    (effects (font (size 0.8 0.8) (thickness 0.2)))
   )
   (gr_text 17 (at 142.0114 94.1324) (layer F.SilkS)
@@
   (segment (start 136.64 70.3072) (end 136.64 68.7952) (width 0.25) (layer F.Cu) (net 0))
   (segment (start 137.4228 68.0124) (end 138.1872 68.0124) (width 0.25) (layer F.Cu) (net 0) (status 20))
-  (segment (start 136.64 68.7952) (end 137.4228 68.0124) (width 0.25) (layer F.Cu) (net 0))
   (segment (start 136.64 72.022) (end 136.64 70.3072) (width 0.25) (layer F.Cu) (net 0) (status 10))
   (segment (start 136.64 70.3072) (end 136.64 70.2176) (width 0.25) (layer F.Cu) (net 0))
@@
   (segment (start 132.6896 72.5932) (end 132.6896 61.5696) (width 0.25) (layer F.Cu) (net 0))
   (segment (start 132.7684 72.672) (end 132.6896 72.5932) (width 0.25) (layer F.Cu) (net 0))
+  (via (at 140.4112 65.7098) (size 0.6) (drill 0.4) (layers F.Cu B.Cu) (net 0))
+  (via (at 136.779 67.818) (size 0.6) (drill 0.4) (layers F.Cu B.Cu) (net 0))
+  (segment (start 139.703 65.7098) (end 140.4112 65.7098) (width 0.25) (layer F.Cu) (net 0))
+  (segment (start 139.5872 65.8256) (end 139.703 65.7098) (width 0.25) (layer F.Cu) (net 0))
+  (segment (start 136.779 68.242264) (end 136.779 67.818) (width 0.25) (layer F.Cu) (net 0))
+  (segment (start 136.964336 68.4276) (end 136.779 68.242264) (width 0.25) (layer F.Cu) (net 0))
+  (segment (start 137.0076 68.4276) (end 136.964336 68.4276) (width 0.25) (layer F.Cu) (net 0))
+  (segment (start 137.0076 68.4276) (end 137.4228 68.0124) (width 0.25) (layer F.Cu) (net 0))
+  (segment (start 136.64 68.7952) (end 137.0076 68.4276) (width 0.25) (layer F.Cu) (net 0))
+  (segment (start 140.835464 65.7098) (end 140.860864 65.7352) (width 0.25) (layer B.Cu) (net 0))
+  (segment (start 140.4112 65.7098) (end 140.835464 65.7098) (width 0.25) (layer B.Cu) (net 0))
+  (segment (start 140.860864 65.7352) (end 141.732 65.7352) (width 0.25) (layer B.Cu) (net 0))
+  (segment (start 141.732 65.7352) (end 141.732 68.199) (width 0.25) (layer B.Cu) (net 0))
+  (segment (start 142.113 68.58) (end 144.78 68.58) (width 0.25) (layer B.Cu) (net 0))
+  (segment (start 141.732 68.199) (end 142.113 68.58) (width 0.25) (layer B.Cu) (net 0))
+  (segment (start 136.779 67.818) (end 136.354736 67.818) (width 0.25) (layer B.Cu) (net 0))
+  (segment (start 143.3068 66.04) (end 144.78 66.04) (width 0.25) (layer B.Cu) (net 0))
+  (segment (start 136.354736 67.818) (end 136.0424 67.505664) (width 0.25) (layer B.Cu) (net 0))
+  (segment (start 136.398 64.9732) (end 142.24 64.9732) (width 0.25) (layer B.Cu) (net 0))
+  (segment (start 136.0424 67.505664) (end 136.0424 65.3288) (width 0.25) (layer B.Cu) (net 0))
+  (segment (start 136.0424 65.3288) (end 136.398 64.9732) (width 0.25) (layer B.Cu) (net 0))
+  (segment (start 142.24 64.9732) (end 143.3068 66.04) (width 0.25) (layer B.Cu) (net 0))
 )
