File: pcb/ftl-12s-rfm-sandwich.kicad_pcb (KiCad board)
At the start: 2 copper layers, 38.1 x 29 mm, 12 parts

Commit message: lora12 2019-Apr2
Parts:
- added 3535: 3535, ws2812:3535, F.Cu at (142.4, 87.0)
- added USB: QFN-16-1EP_3x3mm_Pitch0.5mm, Housings_DFN_QFN:QFN-16-1EP_3x3mm_Pitch0.5mm, F.Cu at (151.1, 86.5)
- VDR1, VDR2: value R_0603_HandSoldering -> R_Axial_DIN0204_L3.6mm_D1.6mm_P1.90mm_Vertical; footprint Resistors_SMD:R_0603_HandSoldering -> Resistors_ThroughHole:R_Axial_DIN0204_L3.6mm_D1.6mm_P1.90mm_Vertical
- moved VREG 7.95 mm to (133.9, 86.5)
- moved VDR1 7.57 mm to (124.5, 105.3), turned to 0 degrees
- moved VDR2 6.23 mm to (130.1, 100.4), turned to 90 degrees
- moved REF** 1.00 mm to (156.0, 81.5)
- moved REF** 1.00 mm to (126.0, 81.5)
- moved NEO 0.48 mm to (157.9, 94.2)
- moved MICRO-B_USB 0.13 mm to (141.8, 78.1)
Routing:
- net (no net): track 346.9 -> 454.1 mm, vias 15 -> 25
Other:
- board size 38.1 x 29 mm -> 38 x 29 mm
- board text added: "lora12 2019-Apr2"
- board text added: "|_|0|_| |_|_|0| |0|0|0|"
- board text removed: "lora12 2019-Apr"
