File: pcb/ftl-12s.kicad_pcb (KiCad board)
At the start: 2 copper layers, 44.5 x 32.4 mm, 10 parts, among them U1 ESP-12

Commit message: catchup
Parts:
- removed the REF** at (124.0, 82.2)
- removed the REF** at (157.4, 82.5)
- added REF**: MountingHole_2.5mm, Mounting_Holes:MountingHole_2.5mm, F.Cu at (126.0, 82.2)
- added REF**: MountingHole_2.5mm, Mounting_Holes:MountingHole_2.5mm, F.Cu at (156.0, 82.5)
- moved MICRO-B_USB 7.78 mm to (141.8, 78.3), turned to 180 degrees
- moved PROG 0.55 mm to (122.3, 97.8)
- moved NEOPIX 0.08 mm to (137.5, 105.1)
- turned VREG to 180 degrees
Routing:
- net (no net): track 20.6 -> 82.0 mm, vias 0 -> 1
Other:
- board size 44.5 x 32.4 mm -> 44 x 30 mm

Commit message: 12x with v1410-usb
Parts:
- removed the REF** at (126.0, 82.2)
- removed the REF** at (156.0, 82.5)
- removed SENS: Pin_Header_Straight_1x03_Pitch2.54mm, Pin_Headers:Pin_Header_Straight_1x03_Pitch2.54mm
- removed U1: ESP-12, kicad-ESP8266:ESP-12
- added ?: ESP-12S, kicad-ESP8266:ESP-07S, B.Cu at (141.3, 94.6)
- added IO0: Measurement_Point_Round-TH_Big, Measurement_Points:Measurement_Point_Round-TH_Big, F.Cu at (137.7, 95.3)
- added PHOTO: Resistor_LDR_5x4.1_RM3, Opto-Devices:Resistor_LDR_5x4.1_RM3, F.Cu at (156.0, 93.5)
- added R1 4K: R_Axial_DIN0207_L6.3mm_D2.5mm_P2.54mm_Vertical, Resistors_ThroughHole:R_Axial_DIN0207_L6.3mm_D2.5mm_P2.54mm_Vertical, F.Cu at (156.0, 87.5)
- added REF**: MountingHole_2.5mm, Mounting_Holes:MountingHole_2.5mm, F.Cu at (126.0, 80.8)
- added REF**: MountingHole_2.5mm, Mounting_Holes:MountingHole_2.5mm, F.Cu at (156.0, 80.9)
- added REF**: APA102, apa102:APA102_hand_solder, F.Cu at (149.6, 93.5)
- added USB: QFN-16-1EP_3x3mm_Pitch0.5mm, Housings_DFN_QFN:QFN-16-1EP_3x3mm_Pitch0.5mm, F.Cu at (142.8, 89.3)
- moved TEMP 27.8 mm to (126.1, 87.3)
- moved SWITCH 8.87 mm to (156.0, 97.8)
- moved PROG 3.94 mm to (126.3, 97.8)
- renumbered SENS to TEMP
Routing:
- net (no net): track 82.0 -> 429.9 mm, vias 1 -> 10
Other:
- board size 44 x 30 mm -> 36 x 30 mm
- board text added: "2019-Apr"
- board text added: "donp.org"
- board text added: "ftl-12s"

Commit message: ftl-12s 2019-Apr
Parts:
- removed the USB at (142.8, 89.3)
- added RTS: Measurement_Point_Round-SMD-Pad_Small, Measurement_Points:Measurement_Point_Round-SMD-Pad_Small, F.Cu at (144.2, 93.4)
- added USB: CP2102N-A01-GQFN-20-3x3mm_0.5mm, Housings_DFN_QFN:SiliconLabs_QFN-20-1EP_3x3mm_Pitch0.5mm, F.Cu at (142.7, 89.8)
- VREG: value DFN-6-1EP_3x3mm_Pitch0.95mm -> LD39050PU33R-DFN-6-3x3mm_0.95mm
- renumbered REF** to APA102
Routing:
- net (no net): track 429.9 -> 477.0 mm, vias 10 -> 14
Other:
- board text added: "1"
- board text added: "15 RX"
- board text added: "16 TX"
- board text added: "3.3v"
- board text added: "4 +V"
- board text added: "5 CO"
- board text added: "5.5v"
- board text added: "6 DO"
- board text added: "9 GND"
- board text added: "ADC 2"
- board text added: "CI 2"
- board text added: "CP2102N-A01-GQFN-20 QFN20-3x3mm_0.5mm"
- board text added: "D"
- board text added: "DI 1"
- board text added: "GND"
- board text added: "GND 3"
- board text added: "IO12"
- board text added: "IO13"
- board text added: "IO2"
- board text added: "IO5"
- board text added: "LD39050PU33R DFN-6-3x3mm_0.95mm"
- board text added: "RST 1"
- board text added: "RX"
- board text added: "TX"
- board text added: "VCC 8"

Commit message: Blinky catchup
Routing:
- net (no net): track 477.0 -> 478.1 mm, vias 14 -> 16
Changed lines of the file:
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@@
     (thickness 1.6)
     (drawings 40)
-    (tracks 229)
+    (tracks 234)
     (zones 0)
     (modules 15)
@@
   (segment (start 140.5128 103.2002) (end 140.2842 103.2002) (width 0.25) (layer F.Cu) (net 0))
   (segment (start 140.2842 103.2002) (end 139.7254 102.6414) (width 0.25) (layer F.Cu) (net 0))
-  (segment (start 139.7254 102.6414) (end 139.7254 93.3196) (width 0.25) (layer B.Cu) (net 0))
-  (segment (start 137.9804 91.5746) (end 133.571 91.5746) (width 0.25) (layer B.Cu) (net 0))
-  (segment (start 139.7254 93.3196) (end 137.9804 91.5746) (width 0.25) (layer B.Cu) (net 0))
   (segment (start 144.8816 94.6912) (end 139.573 94.6912) (width 0.25) (layer F.Cu) (net 0))
   (segment (start 146.812 92.7608) (end 144.8816 94.6912) (width 0.25) (layer F.Cu) (net 0))
@@
   (segment (start 144.2212 91.2622) (end 143.998 91.039) (width 0.25) (layer F.Cu) (net 0))
   (segment (start 144.2212 93.3704) (end 144.2212 91.2622) (width 0.25) (layer F.Cu) (net 0))
+  (via (at 135.4836 102.6668) (size 0.8) (drill 0.4) (layers F.Cu B.Cu) (net 0))
+  (segment (start 139.7254 102.6414) (end 135.509 102.6414) (width 0.25) (layer B.Cu) (net 0))
+  (segment (start 135.509 102.6414) (end 135.4836 102.6668) (width 0.25) (layer B.Cu) (net 0))
+  (via (at 135.7376 92.1766) (size 0.8) (drill 0.4) (layers F.Cu B.Cu) (net 0))
+  (segment (start 135.4836 102.6668) (end 135.4836 92.4306) (width 0.25) (layer F.Cu) (net 0))
+  (segment (start 135.4836 92.4306) (end 135.7376 92.1766) (width 0.25) (layer F.Cu) (net 0))
+  (segment (start 135.1356 91.5746) (end 133.571 91.5746) (width 0.25) (layer B.Cu) (net 0))
+  (segment (start 135.7376 92.1766) (end 135.1356 91.5746) (width 0.25) (layer B.Cu) (net 0))
 )
