File: pcb/bicycle/blinky-2019NovB.kicad_pcb (KiCad board)
At the start: 2 copper layers, 24 x 38 mm, 15 parts

Commit message: catchup
Parts:
- removed the ADC at (134.9, 43.8)
- removed USB: CP2102N-A01-GQFN-20-3x3mm_0.5mm, donpdonp:SiliconLabs_USB_CP2102N-QFN-20-1EP_3x3mm_Pitch0.5mm
- added IO: Pin_Header_Straight_1x03_Pitch2.54mm, Pin_Headers:Pin_Header_Straight_1x03_Pitch2.54mm, F.Cu at (134.9, 43.8)
- moved REF** 9.81 mm to (159.2, 56.2)
- moved REF** 9.81 mm to (159.3, 58.7)
- moved REF** 0.97 mm to (134.9, 52.1), turned to 270 degrees
- moved MICRO-B_USB 0.22 mm to (144.0, 73.0)
- renumbered IO to ADC
Routing:
- net (no net): track 0.00 -> 346.6 mm, vias 0 -> 10
Other:
- board text added: "CK"
- board text added: "DA"
- board text added: "RX"
- board text added: "TX"
